Commit message: Changed name of the package folder from schunk to lwa4d

File: res/models/arm_schunk_with_collisions.urdf (robot description, URDF)
Before this commit: robot teodor_2lwa4d, 13 links, 12 joints
Links:
- link right_arm_1_link: geometry collision mesh filename=package://lwa4d/arm_1_link.stl; visual mesh filename=package://lwa4d/arm_1_link.stl
- link right_arm_2_link: geometry collision mesh filename=package://lwa4d/arm_2_link_collision.stl; visual mesh filename=package://lwa4d/arm_2_link.stl
- link right_arm_3_link: geometry collision mesh filename=package://lwa4d/arm_3_link_collision.stl; visual mesh filename=package://lwa4d/arm_3_link.stl
- link right_arm_4_link: geometry collision mesh filename=package://lwa4d/arm_4_link_collision.stl; visual mesh filename=package://lwa4d/arm_4_link.stl
- link right_arm_5_link: geometry collision mesh filename=package://lwa4d/arm_5_link_collision.stl; visual mesh filename=package://lwa4d/arm_5_link.stl
- link right_arm_6_link: geometry collision mesh filename=package://lwa4d/arm_6_link_collision.stl; visual mesh filename=package://lwa4d/arm_6_link.stl
- link right_arm_7_link: geometry collision mesh filename=package://lwa4d/arm_7_link.stl; visual mesh filename=package://lwa4d/arm_7_link.stl
- link right_arm_podest_link: geometry collision mesh filename=package://lwa4d/arm_podest_link.stl; visual mesh filename=package://lwa4d/arm_podest_link.stl
