Commit message: Created a mimic joint between the left and right finger

File: res/models/schunk_with_fetch.urdf (robot description, URDF)
Before this commit: robot teodor_2lwa4d, 16 links, 15 joints
Joints:
- joint l_gripper_finger_joint: mimic (none) -> joint=r_gripper_finger_joint multiplier=1 offset=0
