Commit message: Played around with the values for the fingers of the gripper

File: res/models/schunk_with_pg70.urdf (robot description, URDF)
Before this commit: robot teodor_2lwa4d, 16 links, 15 joints
Joints:
- joint pg70_finger_left_joint: origin xyz=0 0 0.0789 rpy=0 0 0 -> xyz=0 0.035 0.0789 rpy=0 0 0

Commit message: Changed the dimensions and colors of the fingers in the gripper

File: res/models/schunk_with_pg70.urdf (robot description, URDF)
Before this commit: robot teodor_2lwa4d, 16 links, 15 joints
Links:
- added link pg70_finger_right_link, mass 1; collision box size=0.03 0.01 0.1; visual box size=0.03 0.01 0.1
- link pg70_finger_left_link: geometry collision box size=0.03 0.01 0.1; visual box size=0.03 0.01 0.1
Joints:
- added joint pg70_finger_right_joint: type prismatic, parent pg70_palm_link, child pg70_finger_right_link, origin xyz=0 0.015425 0.0789 rpy=0 0 0, axis 0 -1 0, limit lower=-0.001 upper=0.061 effort=10 velocity=2.0, mimic joint=pg70_finger_left_joint multiplier=1 offset=0
- joint pg70_finger_left_joint: origin xyz=0 0.035 0.0789 rpy=0 0 0 -> xyz=0 -0.015425 0.0789 rpy=0 0 0

Commit message: Corrected issues with the base definition. Removed mimic joint for the right finger

File: res/models/schunk_with_pg70.urdf (robot description, URDF)
Before this commit: robot teodor_2lwa4d, 17 links, 16 joints
Links:
- link mount_link: geometry collision box size=0.02 0.6 0.6; visual box size=0.02 0.6 0.6
- link pg70_finger_left_link: mass 1 -> 0.000001; geometry collision box size=0.04 0.01 0.1; visual box size=0.04 0.01 0.1
- link pg70_finger_right_link: mass 1 -> 0.000001; geometry collision box size=0.04 0.01 0.1; visual box size=0.04 0.01 0.1
- link pg70_palm_link: mass 1 -> 0.000001
- link pg70_podest_link: mass 0.01 -> 0.000001
Joints:
- joint pg70_finger_right_joint: mimic joint=pg70_finger_left_joint multiplier=1 offset=0 -> (none)

Commit message: Updated the inertia parameters

File: res/models/schunk_with_pg70.urdf (robot description, URDF)
Before this commit: robot teodor_2lwa4d, 17 links, 16 joints
Links:
- link right_arm_1_link: mass 0.01 -> 3.6
- link right_arm_2_link: mass 0.01 -> 2.0
- link right_arm_3_link: mass 0.01 -> 2.0
- link right_arm_4_link: mass 0.01 -> 1.2
- link right_arm_5_link: mass 0.01 -> 1.2
- link right_arm_6_link: mass 0.01 -> 1.9
- link right_arm_7_link: mass 0.01 -> 0.05
Joints:
- joint right_arm_1_joint: limit lower=-3.12159265359 upper=3.12159265359 effort=2160 velocity=0.43633 -> lower=-3.12159265359 upper=3.12159265359 effort=216 velocity=0.43633
- joint right_arm_2_joint: limit lower=-2.12 upper=2.12 effort=2160 velocity=0.43633 -> lower=-2.12 upper=2.12 effort=216 velocity=0.43633
- joint right_arm_3_joint: limit lower=-3.12159265359 upper=3.12159265359 effort=815 velocity=0.4189 -> lower=-3.12159265359 upper=3.12159265359 effort=81.5 velocity=0.4189
- joint right_arm_4_joint: limit lower=-2.16 upper=2.16 effort=815 velocity=0.4189 -> lower=-2.16 upper=2.16 effort=81.5 velocity=0.4189
- joint right_arm_5_joint: limit lower=-3.12159265359 upper=3.12159265359 effort=207 velocity=0.43633 -> lower=-3.12159265359 upper=3.12159265359 effort=20.7 velocity=0.43633
- joint right_arm_6_joint: limit lower=-2.07 upper=2.07 effort=150 velocity=1.2566 -> lower=-2.07 upper=2.07 effort=15 velocity=1.2566
- joint right_arm_7_joint: limit lower=-2.94 upper=2.94 effort=150 velocity=1.2566 -> lower=-2.94 upper=2.94 effort=15 velocity=1.2566
- joint right_arm_ee_joint: origin xyz=0 0 0.0824 rpy=0 0 0 -> xyz=0 0 0.0824 rpy=0 0 0.0824

Commit message: Added proper values for the gripper

File: res/models/schunk_with_pg70.urdf (robot description, URDF)
Before this commit: robot teodor_2lwa4d, 17 links, 16 joints
Links:
- link pg70_finger_left_link: mass 0.000001 -> 1; geometry collision box size=0.03 0.01 0.07; visual box size=0.03 0.01 0.07
- link pg70_finger_right_link: mass 0.000001 -> 1; geometry collision box size=0.03 0.01 0.07; visual box size=0.03 0.01 0.07
- link pg70_palm_link: mass 0.000001 -> 1
- link pg70_podest_link: mass 0.000001 -> 1
- link right_arm_ee_link: mass 0.01 -> 1
Joints:
- joint pg70_finger_left_joint: origin xyz=0 -0.015425 0.0789 rpy=0 0 0 -> xyz=0 0.035 0.0789 rpy=0 0 0
- joint pg70_finger_right_joint: origin xyz=0 0.015425 0.0789 rpy=0 0 0 -> xyz=0 -0.035 0.0789 rpy=0 0 0

Commit message: Updated mass and inertia for the gripper

File: res/models/schunk_with_pg70.urdf (robot description, URDF)
Before this commit: robot teodor_2lwa4d, 17 links, 16 joints
Links:
- link pg70_finger_left_link: mass 1 -> 0.01
- link pg70_finger_right_link: mass 1 -> 0.01
- link pg70_podest_link: mass 1 -> 0.01
- link right_arm_ee_link: mass 1 -> 0.01
Joints:
- joint pg70_finger_left_joint: limit lower=-0.001 upper=0.061 effort=10 velocity=2.0 -> lower=-0.001 upper=0.0301 effort=10 velocity=0.041
- joint pg70_finger_right_joint: limit lower=-0.001 upper=0.061 effort=10 velocity=2.0 -> lower=-0.001 upper=0.0301 effort=10 velocity=0.041

Commit message: Added gripper values similar to the fetch gripper

File: res/models/schunk_with_pg70.urdf (robot description, URDF)
Before this commit: robot teodor_2lwa4d, 17 links, 16 joints
Joints:
- joint pg70_finger_left_joint: limit lower=-0.001 upper=0.0301 effort=10 velocity=0.041 -> lower=0.0 upper=0.05 effort=60 velocity=0.05
- joint pg70_finger_right_joint: limit lower=-0.001 upper=0.0301 effort=10 velocity=0.041 -> lower=0.0 upper=0.05 effort=60 velocity=0.05

Commit message: Uncommented the mimic joint

File: res/models/schunk_with_pg70.urdf (robot description, URDF)
Before this commit: robot teodor_2lwa4d, 17 links, 16 joints
Joints:
- joint pg70_finger_right_joint: mimic (none) -> joint=pg70_finger_left_joint multiplier=1 offset=0

Commit message: Modified the joint definitions of the gripper to have a zero position with the fingers almost touching each other

File: res/models/schunk_with_pg70.urdf (robot description, URDF)
Before this commit: robot teodor_2lwa4d, 17 links, 16 joints
Joints:
- joint pg70_finger_left_joint: origin xyz=0 0.035 0.0789 rpy=0 0 0 -> xyz=0 0.0055 0.0789 rpy=0 0 0
- joint pg70_finger_right_joint: origin xyz=0 -0.035 0.0789 rpy=0 0 0 -> xyz=0 -0.0055 0.0789 rpy=0 0 0
- joint right_arm_ee_joint: origin xyz=0 0 0.0824 rpy=0 0 0.0824 -> xyz=0 0 0.0824 rpy=0 0 0

Commit message: Added a virtual link to use as an end_effector. It is located between the fingers of the gripper

File: res/models/schunk_with_pg70.urdf (robot description, URDF)
Before this commit: robot teodor_2lwa4d, 17 links, 16 joints
Links:
- added link end_virtual_link, mass 0.001; visual box size=0.01 0.01 0.01
Joints:
- added joint end_virtual_joint: type fixed, parent pg70_palm_link, child end_virtual_link, origin xyz=0 0 0.09 rpy=0 0 0

Commit message: Changed max velocity of the gripper

File: res/models/schunk_with_pg70.urdf (robot description, URDF)
Before this commit: robot teodor_2lwa4d, 18 links, 17 joints
Joints:
- joint pg70_finger_left_joint: limit lower=0.0 upper=0.05 effort=60 velocity=0.05 -> lower=0.0 upper=0.05 effort=60 velocity=0.03
- joint pg70_finger_right_joint: limit lower=0.0 upper=0.05 effort=60 velocity=0.05 -> lower=0.0 upper=0.05 effort=60 velocity=0.03

Commit message: Moved the fingers a bit up

File: res/models/schunk_with_pg70.urdf (robot description, URDF)
Before this commit: robot teodor_2lwa4d, 18 links, 17 joints
Joints:
- joint pg70_finger_left_joint: origin xyz=0 0.0055 0.0789 rpy=0 0 0 -> xyz=0 0.0055 0.0989 rpy=0 0 0
- joint pg70_finger_right_joint: origin xyz=0 -0.0055 0.0789 rpy=0 0 0 -> xyz=0 -0.0055 0.0989 rpy=0 0 0
